Commit message: Add Cartographer mapping and Scout Mini simulation

File: src/scout_ros-master/scout_description/urdf/scout_mini.urdf.xacro (robot description, xacro)
@@ -50,5 +50,5 @@
     <!-- wheel labeled from 0 to 3, conter-clockwise, starting from front right wheel -->
     <!-- motor 1 and 2 (left side) are mechanically installed in a reversed direction -->
-    <xacro:scout_mini_wheel wheel_prefix="front_right">
+    <xacro:scout_mini_wheel wheel_prefix="front_right" axis_xyz="0 0 1">
         <origin xyz="${wheelbase/2} ${-track/2} ${wheel_vertical_offset}" rpy="1.57 0 0" />
     </xacro:scout_mini_wheel>
@@ -59,5 +59,5 @@
         <origin xyz="${-wheelbase/2} ${track/2} ${wheel_vertical_offset}" rpy="-1.57 0 0" />
     </xacro:scout_mini_wheel>
-    <xacro:scout_mini_wheel wheel_prefix="rear_right">
+    <xacro:scout_mini_wheel wheel_prefix="rear_right" axis_xyz="0 0 1">
         <origin xyz="${-wheelbase/2} ${-track/2} ${wheel_vertical_offset}" rpy="1.57 0 0" />
     </xacro:scout_mini_wheel>

File: src/scout_ros-master/scout_description/urdf/scout_mini_wheel.xacro (robot description, xacro)
@@ -1,5 +1,5 @@
 <?xml version="1.0"?>
 <robot xmlns:xacro="http://ros.org/wiki/xacro" name="scout_wheel">
-    <xacro:macro name="scout_mini_wheel" params="wheel_prefix *joint_pose">
+    <xacro:macro name="scout_mini_wheel" params="wheel_prefix axis_xyz:='0 0 -1' *joint_pose">
         <link name="${wheel_prefix}_wheel_link">
             <inertial>
@@ -28,5 +28,5 @@
             <child link="${wheel_prefix}_wheel_link"/>
             <xacro:insert_block name="joint_pose"/>
-            <axis xyz="0 0 -1" rpy="0 0 0" />
+            <axis xyz="${axis_xyz}" rpy="0 0 0" />
         </joint>
     </xacro:macro>

Commit message: Checkpoint Scout mapping deployment and experiments

File: src/scout_ros-master/scout_description/urdf/scout_mini.urdf.xacro (robot description, xacro)
@@ -3,4 +3,5 @@
     <xacro:arg name="robot_namespace" default="/" />
     <xacro:arg name="urdf_extras" default="empty.urdf" />
+    <xacro:arg name="wheel_axis_multiplier" default="1.0" />
     <xacro:include filename="$(find scout_description)/urdf/scout_mini_wheel.xacro" />
     <!-- Variables -->
@@ -15,4 +16,6 @@
     <xacro:property name="wheel_length" value="0.8e-01" />
     <xacro:property name="wheel_radius" value="1.600e-01" />
+    <xacro:property name="wheel_axis_multiplier"
+                    value="${float('$(arg wheel_axis_multiplier)')}" />
     <!-- Base link -->
     <link name="base_link">
@@ -50,14 +53,18 @@
     <!-- wheel labeled from 0 to 3, conter-clockwise, starting from front right wheel -->
     <!-- motor 1 and 2 (left side) are mechanically installed in a reversed direction -->
-    <xacro:scout_mini_wheel wheel_prefix="front_right" axis_xyz="0 0 1">
+    <xacro:scout_mini_wheel wheel_prefix="front_right"
+                            axis_xyz="0 0 ${wheel_axis_multiplier}">
         <origin xyz="${wheelbase/2} ${-track/2} ${wheel_vertical_offset}" rpy="1.57 0 0" />
     </xacro:scout_mini_wheel>
-    <xacro:scout_mini_wheel wheel_prefix="front_left">
+    <xacro:scout_mini_wheel wheel_prefix="front_left"
+                            axis_xyz="0 0 ${-wheel_axis_multiplier}">
         <origin xyz="${wheelbase/2} ${track/2} ${wheel_vertical_offset}" rpy="-1.57 0 0" />
     </xacro:scout_mini_wheel>
-    <xacro:scout_mini_wheel wheel_prefix="rear_left">
+    <xacro:scout_mini_wheel wheel_prefix="rear_left"
+                            axis_xyz="0 0 ${-wheel_axis_multiplier}">
         <origin xyz="${-wheelbase/2} ${track/2} ${wheel_vertical_offset}" rpy="-1.57 0 0" />
     </xacro:scout_mini_wheel>
-    <xacro:scout_mini_wheel wheel_prefix="rear_right" axis_xyz="0 0 1">
+    <xacro:scout_mini_wheel wheel_prefix="rear_right"
+                            axis_xyz="0 0 ${wheel_axis_multiplier}">
         <origin xyz="${-wheelbase/2} ${-track/2} ${wheel_vertical_offset}" rpy="1.57 0 0" />
     </xacro:scout_mini_wheel>
